Commit message: Making the robot wheel to be stationery both in rviz and gazebo

File: src/custom_warehouse_robot_description/urdf/forklift.urdf.xacro (robot description, xacro)
@@ -86,4 +86,6 @@
       <!-- same axis for both wheels = ROS +Y, so positive velocity drives forward -->
       <axis xyz="${sin(model_yaw)} ${cos(model_yaw)} 0"/>
+      <!-- Damping so wheels actually stop when diff-drive commands zero speed -->
+      <dynamics damping="1.0" friction="0.2"/>
     </joint>
   </xacro:macro>

File: src/custom_warehouse_robot_description/urdf/forklift_gazebo.xacro (robot description, xacro)
@@ -20,8 +20,15 @@
     <maxVel>1.5</maxVel>
   </gazebo>
+  <!-- Help ODE joint motors enforce zero wheel speed when idle -->
+  <gazebo reference="left_wheel_joint">
+    <implicitSpringDamper>true</implicitSpringDamper>
+  </gazebo>
+  <gazebo reference="right_wheel_joint">
+    <implicitSpringDamper>true</implicitSpringDamper>
+  </gazebo>
   <gazebo reference="caster_left">
     <material>Gazebo/Grey</material>
-    <mu1>0.01</mu1>
-    <mu2>0.01</mu2>
+    <mu1>0.1</mu1>
+    <mu2>0.1</mu2>
     <kp>1000000.0</kp>
     <kd>100.0</kd>
@@ -29,6 +36,6 @@
   <gazebo reference="caster_right">
     <material>Gazebo/Grey</material>
-    <mu1>0.01</mu1>
-    <mu2>0.01</mu2>
+    <mu1>0.1</mu1>
+    <mu2>0.1</mu2>
     <kp>1000000.0</kp>
     <kd>100.0</kd>
@@ -50,6 +57,7 @@
       <wheel_diameter>0.10</wheel_diameter>
       <!-- Encoder odom from joints (more consistent wheel "ticks"/integration) -->
-      <max_wheel_torque>8.0</max_wheel_torque>
-      <max_wheel_acceleration>1.0</max_wheel_acceleration>
+      <max_wheel_torque>20.0</max_wheel_torque>
+      <!-- 0 = apply target wheel speed immediately (avoids residual ramp creep) -->
+      <max_wheel_acceleration>0.0</max_wheel_acceleration>
       <command_topic>cmd_vel</command_topic>
       <publish_odom>true</publish_odom>

Commit message: Added AMR warehouse simulation environment

File: src/custom_warehouse_robot_description/urdf/forklift.urdf.xacro (robot description, xacro)
@@ -86,6 +86,6 @@
       <!-- same axis for both wheels = ROS +Y, so positive velocity drives forward -->
       <axis xyz="${sin(model_yaw)} ${cos(model_yaw)} 0"/>
-      <!-- Damping so wheels actually stop when diff-drive commands zero speed -->
-      <dynamics damping="1.0" friction="0.2"/>
+      <!-- Damping light enough that diff-drive motors can still accelerate -->
+      <dynamics damping="0.05" friction="0.02"/>
     </joint>
   </xacro:macro>

File: src/custom_warehouse_robot_description/urdf/forklift_gazebo.xacro (robot description, xacro)
@@ -19,11 +19,4 @@
     <minDepth>0.001</minDepth>
     <maxVel>1.5</maxVel>
-  </gazebo>
-  <!-- Help ODE joint motors enforce zero wheel speed when idle -->
-  <gazebo reference="left_wheel_joint">
-    <implicitSpringDamper>true</implicitSpringDamper>
-  </gazebo>
-  <gazebo reference="right_wheel_joint">
-    <implicitSpringDamper>true</implicitSpringDamper>
   </gazebo>
   <gazebo reference="caster_left">
