Commit message: Stabilize sim drive and lidar for warehouse Nav2.
Add rigid swivel casters, idle cmd_vel zeros, and spawn settle reset to stop post-spawn drift; yaw lidar 180° with a 90–270° FOV and chassis self-filter on /scan_filtered.

Co-authored-by: Cursor <cursoragent@cursor.com>

File: src/custom_warehouse_robot_description/urdf/forklift.urdf.xacro (robot description, xacro)
@@ -19,7 +19,9 @@
   <xacro:property name="wheel_r" value="0.05"/>
   <xacro:property name="wheel_w" value="0.045"/>
-  <!-- Casters: axle at y=0.245, z=-0.0481; ground is z=-0.07 -->
+  <!-- Casters: wheel centre + rigid stem pivot (swivel about Z at the rod) -->
   <xacro:property name="caster_y" value="0.245"/>
   <xacro:property name="caster_z" value="-0.0481"/>
+  <!-- Stem/rod mount on chassis — MUST be the swivel axis so the rod stays rigid -->
+  <xacro:property name="caster_stem_z" value="-0.010"/>
   <xacro:property name="caster_r" value="0.0219"/>
   <!-- Fork slider origin (Fusion Slider 48) -->
@@ -86,18 +88,37 @@
       <!-- same axis for both wheels = ROS +Y, so positive velocity drives forward -->
       <axis xyz="${sin(model_yaw)} ${cos(model_yaw)} 0"/>
-      <!-- Damping light enough that diff-drive motors can still accelerate -->
-      <dynamics damping="0.05" friction="0.02"/>
+      <!-- Enough damping to stop free-roll when cmd_vel is zero -->
+      <dynamics damping="0.8" friction="0.15"/>
     </joint>
   </xacro:macro>
-  <!-- Fixed caster: sphere collision. Make it frictionless in the simulator. -->
+  <!-- Swivel caster: yaw about the rigid stem/rod (NOT the wheel centre).
+       Wheel is a fixed offset below the stem so the rod cannot detach. -->
   <xacro:macro name="caster" params="name mesh px">
+    <link name="${name}_yaw">
+      <inertial>
+        <mass value="0.05"/>
+        <inertia ixx="2e-5" iyy="2e-5" izz="2e-5" ixy="0" ixz="0" iyz="0"/>
+      </inertial>
+    </link>
+    <joint name="${name}_swivel_joint" type="continuous">
+      <parent link="chassis"/>
+      <child link="${name}_yaw"/>
+      <origin xyz="${px-p0x} ${caster_y-p0y} ${caster_stem_z-p0z}" rpy="0 0 0"/>
+      <axis xyz="0 0 1"/>
+      <!-- Higher damping: stops settle-kick and keeps stem feeling rigid -->
+      <dynamics damping="1.5" friction="0.2"/>
+    </joint>
     <link name="${name}">
-      <xacro:mesh_visual file="${mesh}" px="${px}" py="${caster_y}" pz="${caster_z}"/>
+      <!-- Mesh authored in Fusion world frame; keep that offset from stem frame -->
+      <visual>
+        <origin xyz="${-px} ${-caster_y} ${-caster_stem_z}" rpy="0 0 0"/>
+        <geometry><mesh filename="${mesh_dir}/${mesh}.stl"/></geometry>
+      </visual>
       <collision>
-        <origin xyz="0 0 0" rpy="0 0 0"/>
+        <origin xyz="0 0 ${caster_z - caster_stem_z}" rpy="0 0 0"/>
         <geometry><sphere radius="${caster_r}"/></geometry>
       </collision>
       <inertial>
-        <origin xyz="0 -0.012 0.0128" rpy="0 0 0"/>
+        <origin xyz="0 0 ${caster_z - caster_stem_z}" rpy="0 0 0"/>
         <mass value="${caster_mass}"/>
         <inertia ixx="${0.4*caster_mass*caster_r*caster_r}" ixy="0" ixz="0"
@@ -106,8 +127,9 @@
       </inertial>
     </link>
+    <!-- Wheel body rigidly bolted to the swivel fork/rod -->
     <joint name="${name}_joint" type="fixed">
-      <parent link="chassis"/>
+      <parent link="${name}_yaw"/>
       <child link="${name}"/>
-      <origin xyz="${px-p0x} ${caster_y-p0y} ${caster_z-p0z}" rpy="0 0 0"/>
+      <origin xyz="0 0 0" rpy="0 0 0"/>
     </joint>
   </xacro:macro>
@@ -162,6 +184,6 @@
   </joint>
   <!-- ================= LIDAR =================
-       lidar_base holds the mesh (Fusion-aligned); lidar_link is the ROS-aligned
-       sensor frame. Move lidar_link up/down to the real scan plane if needed. -->
+       Rotate the FULL mesh assembly 180° yaw (housing + mounting sticks together).
+       lidar_link keeps Fusion→ROS align relative to that flipped mesh. -->
   <link name="lidar_base">
     <xacro:mesh_visual file="lidar_link" px="0.2093" py="-0.1107" pz="0.3437"/>
@@ -175,5 +197,5 @@
     <parent link="chassis"/>
     <child link="lidar_base"/>
-    <origin xyz="${0.2093-p0x} ${-0.1107-p0y} ${0.3437-p0z}" rpy="0 0 0"/>
+    <origin xyz="${0.2093-p0x} ${-0.1107-p0y} ${0.3437-p0z}" rpy="0 0 ${pi}"/>
   </joint>
   <link name="lidar_link"/>

File: src/custom_warehouse_robot_description/urdf/forklift_gazebo.xacro (robot description, xacro)
@@ -22,6 +22,6 @@
   <gazebo reference="caster_left">
     <material>Gazebo/Grey</material>
-    <mu1>0.1</mu1>
-    <mu2>0.1</mu2>
+    <mu1>0.02</mu1>
+    <mu2>0.02</mu2>
     <kp>1000000.0</kp>
     <kd>100.0</kd>
@@ -29,6 +29,6 @@
   <gazebo reference="caster_right">
     <material>Gazebo/Grey</material>
-    <mu1>0.1</mu1>
-    <mu2>0.1</mu2>
+    <mu1>0.02</mu1>
+    <mu2>0.02</mu2>
     <kp>1000000.0</kp>
     <kd>100.0</kd>
@@ -71,6 +71,15 @@
       <joint_name>right_wheel_joint</joint_name>
       <joint_name>fork_lift_joint</joint_name>
+      <joint_name>caster_left_swivel_joint</joint_name>
+      <joint_name>caster_right_swivel_joint</joint_name>
     </plugin>
   </gazebo>
+  <!-- Scan FOV matches config/lidar.yaml (90° → 270°) -->
+  <xacro:property name="lidar_samples" value="360"/>
+  <xacro:property name="lidar_min_angle" value="${pi/2}"/>
+  <xacro:property name="lidar_max_angle" value="${3.0 * pi / 2.0}"/>
+  <xacro:property name="lidar_range_min" value="0.40"/>
+  <xacro:property name="lidar_range_max" value="25.0"/>
+  <xacro:property name="lidar_update_rate" value="15.0"/>
   <gazebo reference="lidar_link">
     <sensor name="laser_scanner" type="ray">
@@ -78,19 +87,18 @@
       <always_on>true</always_on>
       <visualize>false</visualize>
-      <update_rate>15.0</update_rate>
+      <update_rate>${lidar_update_rate}</update_rate>
       <ray>
         <scan>
           <horizontal>
-            <!-- 275° FOV centered forward (±137.5°) -->
-            <samples>550</samples>
+            <samples>${lidar_samples}</samples>
             <resolution>1</resolution>
-            <min_angle>-2.3998277</min_angle>
-            <max_angle>2.3998277</max_angle>
+            <min_angle>${lidar_min_angle}</min_angle>
+            <max_angle>${lidar_max_angle}</max_angle>
           </horizontal>
         </scan>
         <range>
           <!-- Keep min range above robot body to avoid self-hits as false obstacles -->
-          <min>0.30</min>
-          <max>25.0</max>
+          <min>${lidar_range_min}</min>
+          <max>${lidar_range_max}</max>
           <resolution>0.01</resolution>
         </range>
